File: KiCad/PCB336/PCB336.kicad_sch (KiCad schematic)
At the start: 0 parts

Commit message: Filament Pagina in lavorazione
Other:
- company: (none) -> METALTRONICA
- title: (none) -> PCB/25-336-1
Changed lines of the file:
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@@
 	(generator_version "10.0")
 	(paper "A4")
+	(title_block
+		(title "PCB/25-336-1")
+		(rev "0")
+		(company "METALTRONICA")
+	)
 	(sheet_instances
 		(path "/"
