File: KiCad/PCB336/PCB336.kicad_pcb (KiCad board)
At the start: 2 copper layers, 40 parts, among them IC1 NJM78L12UA-TE1, IC2 NJM79L12SU3-TE1, IC3 TSR_0.5-2450, J1 39-29-9043, U1 NCP1117ST33T3G

Commit message: Filament Pagina in lavorazione
Parts:
- added C18: 100nF, Capacitor_SMD:C_0805_2012Metric_Pad1.18x1.45mm_HandSolder, F.Cu at (30.3, 82.5)
- added C19: 100nF, Capacitor_SMD:C_0805_2012Metric_Pad1.18x1.45mm_HandSolder, F.Cu at (30.3, 85.5)
- added C20: 100nF, Capacitor_SMD:C_0805_2012Metric_Pad1.18x1.45mm_HandSolder, F.Cu at (30.3, 88.5)
- added C21: 100nF, Capacitor_SMD:C_0805_2012Metric_Pad1.18x1.45mm_HandSolder, F.Cu at (30.3, 91.5)
- added C22: 100nF, Capacitor_SMD:C_0805_2012Metric_Pad1.18x1.45mm_HandSolder, F.Cu at (30.3, 94.5)
- added C23: 100nF, Capacitor_SMD:C_0805_2012Metric_Pad1.18x1.45mm_HandSolder, F.Cu at (35.1, 82.5)
- added C24: 100nF, Capacitor_SMD:C_0805_2012Metric_Pad1.18x1.45mm_HandSolder, F.Cu at (35.1, 85.5)
- added C25: 100nF, Capacitor_SMD:C_0805_2012Metric_Pad1.18x1.45mm_HandSolder, F.Cu at (35.1, 88.5)
- added C26: 4u7, Capacitor_SMD:C_0805_2012Metric_Pad1.18x1.45mm_HandSolder, F.Cu at (35.1, 91.5)
- added C29: 10uF, Capacitor_SMD:C_0805_2012Metric_Pad1.18x1.45mm_HandSolder, F.Cu at (35.1, 94.5)
- added Q1: 2N7002LT1G, Package_TO_SOT_SMD:SOT-23, F.Cu at (25.5, 83.2)
- added Q2: 2N7002LT1G, Package_TO_SOT_SMD:SOT-23, F.Cu at (25.5, 87.7)
- added Q3: 2N7002LT1G, Package_TO_SOT_SMD:SOT-23, F.Cu at (25.5, 92.1)
- added Q4: 2N7002LT1G, Package_TO_SOT_SMD:SOT-23, F.Cu at (25.5, 96.6)
- added Q5: 2N7002LT1G, Package_TO_SOT_SMD:SOT-23, F.Cu at (25.5, 101.0)
- added Q6: 2N7002LT1G, Package_TO_SOT_SMD:SOT-23, F.Cu at (25.5, 105.5)
- added R10: 680R, Resistor_SMD:R_0603_1608Metric_Pad0.98x0.95mm_HandSolder, F.Cu at (44.1, 99.1)
- added R11: 33K, Resistor_SMD:R_0603_1608Metric_Pad0.98x0.95mm_HandSolder, F.Cu at (44.1, 101.6)
- added R12: 680R, Resistor_SMD:R_0603_1608Metric_Pad0.98x0.95mm_HandSolder, F.Cu at (44.1, 104.1)
- added R13: 33K, Resistor_SMD:R_0603_1608Metric_Pad0.98x0.95mm_HandSolder, F.Cu at (44.1, 106.6)
- added R14: 680R, Resistor_SMD:R_0603_1608Metric_Pad0.98x0.95mm_HandSolder, F.Cu at (48.4, 96.6)
- added R15: 33K, Resistor_SMD:R_0603_1608Metric_Pad0.98x0.95mm_HandSolder, F.Cu at (48.4, 99.1)
- added R16: 680R, Resistor_SMD:R_0603_1608Metric_Pad0.98x0.95mm_HandSolder, F.Cu at (48.4, 101.6)
- added R17: 33K, Resistor_SMD:R_0603_1608Metric_Pad0.98x0.95mm_HandSolder, F.Cu at (48.4, 104.1)
- added R18: 680R, Resistor_SMD:R_0603_1608Metric_Pad0.98x0.95mm_HandSolder, F.Cu at (48.4, 106.6)
- added R4: 10K, Resistor_SMD:R_0603_1608Metric_Pad0.98x0.95mm_HandSolder, F.Cu at (39.7, 96.6)
- added R5: 330R, Resistor_SMD:R_0603_1608Metric_Pad0.98x0.95mm_HandSolder, F.Cu at (39.7, 99.1)
- added R6: 1K, Resistor_SMD:R_0603_1608Metric_Pad0.98x0.95mm_HandSolder, F.Cu at (39.7, 101.6)
- added R7: 680R, Resistor_SMD:R_0603_1608Metric_Pad0.98x0.95mm_HandSolder, F.Cu at (39.7, 104.1)
- added R8: 33K, Resistor_SMD:R_0603_1608Metric_Pad0.98x0.95mm_HandSolder, F.Cu at (39.7, 106.6)
- added R9: 33K, Resistor_SMD:R_0603_1608Metric_Pad0.98x0.95mm_HandSolder, F.Cu at (44.1, 96.6)
- added U2: ATSAME51J20A-A, Package_QFP:TQFP-64_10x10mm_P0.5mm, F.Cu at (44.7, 88.2)

Commit message: Avanzamenti in Agosto
Parts:
- removed TP2: RED, MET:TP_5001
- added C27: 10nF, Capacitor_SMD:C_0805_2012Metric_Pad1.18x1.45mm_HandSolder, F.Cu at (38.7, 94.0)
- added C28: 100nF, Capacitor_SMD:C_0805_2012Metric_Pad1.18x1.45mm_HandSolder, F.Cu at (38.7, 97.0)
- added C30: 10uF, Capacitor_SMD:C_1206_3216Metric_Pad1.33x1.80mm_HandSolder, F.Cu at (92.2, 62.6)
- added C31: 1uF, Capacitor_SMD:C_1206_3216Metric_Pad1.33x1.80mm_HandSolder, F.Cu at (92.2, 65.9)
- added C32: 1uF, Capacitor_SMD:C_1206_3216Metric_Pad1.33x1.80mm_HandSolder, F.Cu at (92.2, 69.3)
- added C33: 1uF, Capacitor_SMD:C_1206_3216Metric_Pad1.33x1.80mm_HandSolder, F.Cu at (92.2, 72.6)
- added C34: 100pF, Capacitor_SMD:C_0603_1608Metric_Pad1.08x0.95mm_HandSolder, F.Cu at (43.2, 87.7)
- added C35: 1uF, Capacitor_SMD:C_1206_3216Metric_Pad1.33x1.80mm_HandSolder, F.Cu at (92.2, 76.0)
- added C36: 1uF, Capacitor_SMD:C_1206_3216Metric_Pad1.33x1.80mm_HandSolder, F.Cu at (92.2, 79.3)
- added C37: 470pF, Capacitor_SMD:C_0603_1608Metric_Pad1.08x0.95mm_HandSolder, F.Cu at (43.2, 90.2)
- added C38: 1uF, Capacitor_SMD:C_1206_3216Metric_Pad1.33x1.80mm_HandSolder, F.Cu at (92.2, 82.7)
- added D4: BLUE, MET:LED_0805, F.Cu at (33.4, 106.0)
- added D5: RED, MET:LED_0805, F.Cu at (33.4, 109.1)
- added D6: YELLOW, MET:LED_0805, F.Cu at (33.4, 112.2)
- added D7: YELLOW, MET:LED_0805, F.Cu at (37.9, 106.0)
- added D8: YELLOW, MET:LED_0805, F.Cu at (37.9, 109.1)
- added D9: YELLOW, MET:LED_0805, F.Cu at (37.9, 112.2)
- added IC4: XR2206CP-F, MET:XR2206CP, F.Cu at (100.7, 72.3)
- added IC5: LM1458MX_NOPB, MET:SOIC_LM1458M, F.Cu at (110.4, 71.4)
- added J2: 61200621621, MET:uCProg_61200621621, F.Cu at (46.9, 110.6)
- added L2: BLM18BD102SN1D, MET:BLM18SP221SN1B, F.Cu at (116.7, 69.4)
- added L3: BLM18BD102SN1D, MET:BLM18SP221SN1B, F.Cu at (116.7, 71.9)
- added R19: 5K6, Resistor_SMD:R_0603_1608Metric_Pad0.98x0.95mm_HandSolder, F.Cu at (51.9, 95.2)
- added R20: 5K6, Resistor_SMD:R_0603_1608Metric_Pad0.98x0.95mm_HandSolder, F.Cu at (51.9, 97.7)
- added R21: 5K6, Resistor_SMD:R_0603_1608Metric_Pad0.98x0.95mm_HandSolder, F.Cu at (51.9, 100.2)
- added R22: 5K6, Resistor_SMD:R_0603_1608Metric_Pad0.98x0.95mm_HandSolder, F.Cu at (51.9, 102.7)
- added R23: 220R, Resistor_SMD:R_0603_1608Metric_Pad0.98x0.95mm_HandSolder, F.Cu at (56.3, 87.7)
- added R24: 10K, Resistor_SMD:R_0603_1608Metric_Pad0.98x0.95mm_HandSolder, F.Cu at (56.3, 90.2)
- added R25: 2K, Resistor_SMD:R_0603_1608Metric_Pad0.98x0.95mm_HandSolder, F.Cu at (56.3, 92.7)
- added R26: 2K, Resistor_SMD:R_0603_1608Metric_Pad0.98x0.95mm_HandSolder, F.Cu at (56.3, 95.2)
- added R27: 1K, Resistor_SMD:R_0603_1608Metric_Pad0.98x0.95mm_HandSolder, F.Cu at (56.3, 97.7)
- added R28: 56K, Resistor_SMD:R_0603_1608Metric_Pad0.98x0.95mm_HandSolder, F.Cu at (56.3, 100.2)
- added RV1: 20K, Potentiometer_THT:Potentiometer_Bourns_3296W_Vertical, F.Cu at (114.3, 77.8)
- added TP10: 5002, MET:TP_5001, F.Cu at (81.5, 110.1)
- added TP8: 5002, MET:TP_5001, F.Cu at (81.5, 102.7)
- added TP9: 5000, MET:TP_5001, F.Cu at (81.5, 106.4)
- added U3: PCB319-2, MET:PCB319-2, F.Cu at (42.5, 83.7)
- TP1, TP4, TP5, TP6, TP7: value RED -> 5000
- TP3: value BLACK -> 5001
- moved Q4 107.9 mm to (116.7, 39.0)
- moved Q5 107.9 mm to (116.7, 43.4)
- moved Q1 107.9 mm to (116.7, 25.6)
- moved Q2 107.9 mm to (116.7, 30.1)
- moved Q3 107.9 mm to (116.7, 34.5)
- moved Q6 107.9 mm to (116.7, 47.9)
- moved L1 84.2 mm to (109.6, 64.5)
- moved U1 80.5 mm to (114.2, 106.9)
- moved D1 73.7 mm to (28.9, 106.0)
- moved D2 73.7 mm to (28.9, 109.1)
- moved D3 73.7 mm to (28.9, 112.2)
- moved C1 73.2 mm to (92.0, 88.9)
- moved C3 73.2 mm to (101.2, 88.9)
- moved C5 73.2 mm to (110.4, 88.9)
- moved J1 73.2 mm to (101.3, 112.3)
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
Commit message: Completato Filament e Monitor
Parts:
- added C39: 100nF, Capacitor_SMD:C_0805_2012Metric_Pad1.18x1.45mm_HandSolder, F.Cu at (118.2, 77.6)
- added C40: 33uF, MET:WCAP-HTG5_D8_H9_P3.5, F.Cu at (79.0, 91.2)
- added C41: 33uF, MET:WCAP-HTG5_D8_H9_P3.5, F.Cu at (79.0, 100.3)
- added C42: 100uF, Capacitor_THT:CP_Radial_D18.0mm_P7.50mm, F.Cu at (35.1, 96.3)
- added C43: 100uF, Capacitor_THT:CP_Radial_D18.0mm_P7.50mm, F.Cu at (35.1, 115.9)
- added C44: 10uF, Capacitor_SMD:C_1206_3216Metric_Pad1.33x1.80mm_HandSolder, F.Cu at (94.1, 114.3)
- added C45: 100nF, Capacitor_SMD:C_0805_2012Metric_Pad1.18x1.45mm_HandSolder, F.Cu at (123.0, 62.5)
- added C46: 100nF, Capacitor_SMD:C_0805_2012Metric_Pad1.18x1.45mm_HandSolder, F.Cu at (123.0, 65.5)
- added C47: 100nF, Capacitor_SMD:C_0805_2012Metric_Pad1.18x1.45mm_HandSolder, F.Cu at (123.0, 68.5)
- added C48: 47nF, Capacitor_SMD:C_0805_2012Metric_Pad1.18x1.45mm_HandSolder, F.Cu at (123.0, 71.5)
- added C49: 1uF, Capacitor_SMD:C_1206_3216Metric_Pad1.33x1.80mm_HandSolder, F.Cu at (94.1, 117.7)
- added C50: 100nF, Capacitor_SMD:C_0805_2012Metric_Pad1.18x1.45mm_HandSolder, F.Cu at (123.0, 74.5)
- added C51: 100nF, Capacitor_SMD:C_0805_2012Metric_Pad1.18x1.45mm_HandSolder, F.Cu at (123.0, 77.6)
- added D10: SK56C, MET:SK56C, F.Cu at (132.3, 27.4)
- added D11: SK56C, MET:SK56C, F.Cu at (132.3, 35.2)
- added D12: BAT754S,215, MET:BAT754S,215, F.Cu at (121.4, 81.3)
- added D13: BAT754S,215, MET:BAT754S,215, F.Cu at (121.4, 85.9)
- added D14: 1N4148W, Diode_SMD:D_SOD-123, F.Cu at (111.0, 104.1)
- added D15: 1N4148W, Diode_SMD:D_SOD-123, F.Cu at (111.0, 107.4)
- added D16: 1N4148W, Diode_SMD:D_SOD-123, F.Cu at (111.0, 110.8)
- added D17: 1N4148W, Diode_SMD:D_SOD-123, F.Cu at (111.0, 114.1)
- added D18: 1N4148W, Diode_SMD:D_SOD-123, F.Cu at (111.0, 117.5)
- added D19: 1N4148W, Diode_SMD:D_SOD-123, F.Cu at (111.0, 120.8)
- added D20: 1N4148W, Diode_SMD:D_SOD-123, F.Cu at (116.7, 104.1)
- added D21: 1N4148W, Diode_SMD:D_SOD-123, F.Cu at (116.7, 107.4)
- added D22: 1N4148W, Diode_SMD:D_SOD-123, F.Cu at (116.7, 110.8)
- added D23: 1N4148W, Diode_SMD:D_SOD-123, F.Cu at (116.7, 114.1)
- added D24: 1N4148W, Diode_SMD:D_SOD-123, F.Cu at (116.7, 117.5)
- added IC6: MCP4821-E/MS, MET:MCP4821_EMS, F.Cu at (104.7, 58.0)
- added IC7: LM358BAIDR, MET:LM358BAIDR, F.Cu at (132.4, 99.0)
- added J3: Piazzolato, Connector_PinSocket_2.54mm:PinSocket_1x05_P2.54mm_Vertical, F.Cu at (135.6, 104.7)
- added JP1: SolderJumper_2_Bridged, Jumper:SolderJumper-2_P1.3mm_Bridged2Bar_Pad1.0x1.5mm, F.Cu at (133.5, 81.5)
- added Q7: 2N7002LT1G, Package_TO_SOT_SMD:SOT-23, F.Cu at (104.4, 123.2)
- added R29: 2K2, Resistor_SMD:R_0603_1608Metric_Pad0.98x0.95mm_HandSolder, F.Cu at (59.5, 123.8)
- added R30: 4K7, Resistor_SMD:R_1206_3216Metric_Pad1.30x1.75mm_HandSolder, F.Cu at (128.4, 81.4)
- added R31: 4K7, Resistor_SMD:R_1206_3216Metric_Pad1.30x1.75mm_HandSolder, F.Cu at (128.4, 84.7)
- added R32: 200R, Resistor_SMD:R_0603_1608Metric_Pad0.98x0.95mm_HandSolder, F.Cu at (59.5, 126.3)
- added R33: 200R, Resistor_SMD:R_0603_1608Metric_Pad0.98x0.95mm_HandSolder, F.Cu at (59.5, 128.8)
- added R34: 10K, Resistor_SMD:R_0603_1608Metric_Pad0.98x0.95mm_HandSolder, F.Cu at (63.8, 106.2)
- added R35: 87K, Resistor_SMD:R_0603_1608Metric_Pad0.98x0.95mm_HandSolder, F.Cu at (63.8, 108.7)
- added R36: 10K, Resistor_SMD:R_0603_1608Metric_Pad0.98x0.95mm_HandSolder, F.Cu at (63.8, 111.2)
- added R37: 10K, Resistor_SMD:R_0603_1608Metric_Pad0.98x0.95mm_HandSolder, F.Cu at (63.8, 113.7)
- added R38: 10K, Resistor_SMD:R_0603_1608Metric_Pad0.98x0.95mm_HandSolder, F.Cu at (63.8, 116.2)
- added R39: 10K, Resistor_SMD:R_0603_1608Metric_Pad0.98x0.95mm_HandSolder, F.Cu at (63.8, 118.8)
- added R40: 39K, Resistor_SMD:R_0603_1608Metric_Pad0.98x0.95mm_HandSolder, F.Cu at (63.8, 121.3)
- added R41: 27K, Resistor_SMD:R_0603_1608Metric_Pad0.98x0.95mm_HandSolder, F.Cu at (63.8, 123.8)
- added R42: 10K, Resistor_SMD:R_0603_1608Metric_Pad0.98x0.95mm_HandSolder, F.Cu at (63.8, 126.3)
- added R43: 10K, Resistor_SMD:R_0603_1608Metric_Pad0.98x0.95mm_HandSolder, F.Cu at (63.8, 128.8)
- added R44: 4K7, Resistor_SMD:R_0603_1608Metric_Pad0.98x0.95mm_HandSolder, F.Cu at (68.2, 106.2)
- added R45: 5K6, Resistor_SMD:R_0603_1608Metric_Pad0.98x0.95mm_HandSolder, F.Cu at (68.2, 108.7)
- added R46: 18K, Resistor_SMD:R_0603_1608Metric_Pad0.98x0.95mm_HandSolder, F.Cu at (68.2, 111.2)
- added R47: 4K7, Resistor_SMD:R_0603_1608Metric_Pad0.98x0.95mm_HandSolder, F.Cu at (68.2, 113.7)
- added R48: 10K, Resistor_SMD:R_0603_1608Metric_Pad0.98x0.95mm_HandSolder, F.Cu at (68.2, 116.2)
- added R49: 100K, Resistor_SMD:R_0603_1608Metric_Pad0.98x0.95mm_HandSolder, F.Cu at (68.2, 118.8)
- added R50: 100K, Resistor_SMD:R_0603_1608Metric_Pad0.98x0.95mm_HandSolder, F.Cu at (68.2, 121.3)
- added R51: 10K, Resistor_SMD:R_0603_1608Metric_Pad0.98x0.95mm_HandSolder, F.Cu at (68.2, 123.8)
- added R52: 10K, Resistor_SMD:R_0603_1608Metric_Pad0.98x0.95mm_HandSolder, F.Cu at (68.2, 126.3)
- added R53: 87K, Resistor_SMD:R_0603_1608Metric_Pad0.98x0.95mm_HandSolder, F.Cu at (68.2, 128.8)
- added R54: 5K6, Resistor_SMD:R_0603_1608Metric_Pad0.98x0.95mm_HandSolder, F.Cu at (72.5, 106.2)
- added R55: 4K7, Resistor_SMD:R_0603_1608Metric_Pad0.98x0.95mm_HandSolder, F.Cu at (72.5, 108.7)
- added R56: 10K, Resistor_SMD:R_0603_1608Metric_Pad0.98x0.95mm_HandSolder, F.Cu at (72.5, 111.2)
- added R57: 22K, Resistor_SMD:R_0603_1608Metric_Pad0.98x0.95mm_HandSolder, F.Cu at (72.5, 113.7)
- added R59: 10K, Resistor_SMD:R_0603_1608Metric_Pad0.98x0.95mm_HandSolder, F.Cu at (72.5, 116.2)
- added R60: 100K, Resistor_SMD:R_0603_1608Metric_Pad0.98x0.95mm_HandSolder, F.Cu at (72.5, 118.8)
- added RV2: 5K, Potentiometer_THT:Potentiometer_Bourns_3296W_Vertical, F.Cu at (82.8, 114.5)
- added T1: TF-108, MET:TF-108, F.Cu at (110.4, 27.5)
- added TP11: 5002, MET:TP_5001, F.Cu at (131.0, 77.8)
- added TP12: 5001, MET:TP_5001, F.Cu at (134.7, 62.9)
- added TP13: 5002, MET:TP_5001, F.Cu at (134.7, 66.6)
- added TP14: 5002, MET:TP_5001, F.Cu at (134.7, 70.3)
- moved J2 97.2 mm to (121.2, 47.9)
- moved D3 94.1 mm to (121.9, 126.4)
- moved D6 94.1 mm to (126.4, 126.4)
- moved D9 94.1 mm to (130.9, 126.4)
- moved D1 94.1 mm to (121.9, 120.2)
- moved D2 94.1 mm to (121.9, 123.3)
- moved D4 94.1 mm to (126.4, 120.2)
- moved D5 94.1 mm to (126.4, 123.3)
- moved D7 94.1 mm to (130.9, 120.2)
- moved D8 94.1 mm to (130.9, 123.3)
- moved Q2 90.4 mm to (99.5, 118.8)
- moved Q3 90.4 mm to (99.5, 123.2)
- moved Q4 90.4 mm to (99.5, 127.7)
- moved Q1 90.4 mm to (99.5, 114.3)
- moved C10 83.5 mm to (108.6, 65.5)
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Connections:
- net /uController/uC_FILFREQ renamed /uController/uC_IFREQ_ANL
- net /uController/uC_VFILx5_ANL renamed /uController/uC_VFIL_ANL
- C1 pad 2: GND1 -> GNDPWR
- C2 pad 2: GND1 -> GNDPWR
- C3 pad 2: GND1 -> GNDPWR
- C38 pad 2: Net-(C38-Pad2) -> /FilamentControl/vamp
- C4 pad 1: GND1 -> GNDPWR
- C5 pad 1: GND1 -> GNDPWR
- C6 pad 1: GND1 -> GNDPWR
- FL1 pad 4: GND1 -> GNDPWR
- FL1 pad 5: GND1 -> GNDPWR
- FL1 pad 6: GND1 -> GNDPWR
- FL2 pad 2: GND1 -> GNDPWR
- IC5 pad 5: unconnected-(IC5-+B-Pad5) -> GND
- IC5 pad 6: unconnected-(IC5--B-Pad6) -> Net-(IC5--B)
- IC5 pad 7: unconnected-(IC5-OB-Pad7) -> /FilamentControl/MONITOR_24VNEG
- R28 pad 1: Net-(C38-Pad2) -> /FilamentControl/vamp
- U2 pad 9: /uController/uC_VFILx15_ANL -> unconnected-(U2-PB06-Pad9)
- U3 pad 1: unconnected-(U3-+T-Pad1) -> /FilamentControl/MONITOR_TAMP
- U3 pad 10: unconnected-(U3-B--Pad10) -> -24V
- U3 pad 11: unconnected-(U3-B+-Pad11) -> +24V
- U3 pad 12: unconnected-(U3-Out-Pad12) -> Net-(D10-A)
- U3 pad 13: unconnected-(U3-Out2-Pad13) -> Net-(D10-A)
- U3 pad 2: unconnected-(U3--T-Pad2) -> GND
- U3 pad 3: unconnected-(U3-In-Pad3) -> /FilamentControl/vamp
- U3 pad 5: unconnected-(U3-GNDP-Pad5) -> GNDPWR
- U3 pad 6: unconnected-(U3-nc2-Pad6) -> -24V

Commit message: Completato schematico, e ERC Iniziato piazzamento
Parts:
- added C52: 100nF, Capacitor_SMD:C_0805_2012Metric_Pad1.18x1.45mm_HandSolder, F.Cu at (-43.5, 56.2)
- added C53: 100nF, Capacitor_SMD:C_0805_2012Metric_Pad1.18x1.45mm_HandSolder, F.Cu at (-43.5, 59.2)
- added C54: 100nF, Capacitor_SMD:C_0805_2012Metric_Pad1.18x1.45mm_HandSolder, F.Cu at (-43.5, 62.2)
- added C55: 100nF, Capacitor_SMD:C_0805_2012Metric_Pad1.18x1.45mm_HandSolder, F.Cu at (-38.7, 38.1)
- added C56: 10nF, Capacitor_SMD:C_0805_2012Metric_Pad1.18x1.45mm_HandSolder, F.Cu at (-38.7, 41.1)
- added C57: 4.7uF, MET:T491C, F.Cu at (-60.5, 46.0)
- added C58: 4.7uF, MET:T491C, F.Cu at (-60.5, 52.2)
- added C59: 470pF, MET:C470pF_WURTH_APC4632X160N, F.Cu at (-111.3, 119.6)
- added C60: 100nF, Capacitor_SMD:C_0805_2012Metric_Pad1.18x1.45mm_HandSolder, F.Cu at (-38.7, 44.1)
- added C61: 100nF, Capacitor_SMD:C_0805_2012Metric_Pad1.18x1.45mm_HandSolder, F.Cu at (-38.7, 47.1)
- added C62: 1uF, Capacitor_SMD:C_1206_3216Metric_Pad1.33x1.80mm_HandSolder, F.Cu at (-40.3, 20.9)
- added C63: 1uF, Capacitor_SMD:C_1206_3216Metric_Pad1.33x1.80mm_HandSolder, F.Cu at (-40.3, 24.3)
- added C64: 1uF, Capacitor_SMD:C_1206_3216Metric_Pad1.33x1.80mm_HandSolder, F.Cu at (-40.3, 27.6)
- added C65: 100nF, Capacitor_SMD:C_0805_2012Metric_Pad1.18x1.45mm_HandSolder, F.Cu at (-38.7, 50.1)
- added C66: 100nF, Capacitor_SMD:C_0805_2012Metric_Pad1.18x1.45mm_HandSolder, F.Cu at (-38.7, 53.2)
- added C67: 4.7uF, MET:T491C, F.Cu at (-60.5, 58.5)
- added C68: 4.7uF, MET:T491C, F.Cu at (-60.5, 64.7)
- added D25: ES1A, MET:ES1A, F.Cu at (-84.7, 62.7)
- added D26: ES1A, MET:ES1A, F.Cu at (-84.7, 67.1)
- added D27: ES1A, MET:ES1A, F.Cu at (-84.7, 71.5)
- added D28: ES1A, MET:ES1A, F.Cu at (-84.7, 75.9)
- added D29: ESDM2032MX4T5G, MET:ESDM2032MX4T5G, F.Cu at (-21.9, 100.2)
- added D30: GREEN, MET:LED_0805, F.Cu at (-89.1, 106.0)
- added D31: GREEN, MET:LED_0805, F.Cu at (-89.1, 109.1)
- added IC10: ADM4857ARZ-REEL7, MET:ADM4857_SOIC, F.Cu at (-21.1, 53.0)
- added IC11: ADM4857ARZ-REEL7, MET:ADM4857_SOIC, F.Cu at (-21.1, 59.5)
- added IC12: MAX22246CAWA_V+, MET:MAX22246_SOIC127P1031X265-8N, F.Cu at (-69.0, 117.7)
- added IC13: TJA1050T_CM,118, MET:TJA1050T_SOIC127P600X175-8N, F.Cu at (-42.6, 32.6)
- added IC14: ESD2CAN24DBZRQ1, MET:ESD2CAN24DBZRQ1, F.Cu at (-15.0, 118.2)
- added IC15: NJM78L05UA-TE1, MET:NJM78L05UA-TE1, F.Cu at (-20.3, 119.2)
- added IC8: ADUM3195BRQZ, MET:SOP64P599X175-16N, F.Cu at (-51.1, 32.7)
- added IC9: ISO6742FDWR, MET:ISO6742FDWR_SOIC, F.Cu at (-108.2, 111.0)
- added J4: MOLEX_172298-1108, MET:MOLEX_172298_1108, F.Cu at (-38.3, 93.2)
- added J5: 105310-2210, MET:1053102210, F.Cu at (-47.1, 89.3)
- added J6: 105310-2210, MET:1053102210, F.Cu at (-47.1, 98.6)
- added J7: 105312-1104, MET:NANOFIT_1053121104, F.Cu at (-38.0, 111.4)
- added J8: 105312-1104, MET:NANOFIT_1053121104, F.Cu at (-25.9, 111.4)
- added K1: 32.21.7.024.4000, MET:322170244000, F.Cu at (-135.0, 71.0)
- added K2: 32.21.7.024.4000, MET:322170244000, F.Cu at (-135.0, 84.2)
- added K3: 32.21.7.024.4000, MET:322170244000, F.Cu at (-135.0, 97.4)
- added K4: 32.21.7.024.4000, MET:322170244000, F.Cu at (-135.0, 110.6)
- added Q10: 2N7002LT1G, Package_TO_SOT_SMD:SOT-23, F.Cu at (-17.2, 74.5)
- added Q11: 2N7002LT1G, Package_TO_SOT_SMD:SOT-23, F.Cu at (-17.2, 79.0)
- added Q8: 2N7002LT1G, Package_TO_SOT_SMD:SOT-23, F.Cu at (-22.1, 83.4)
- added Q9: 2N7002LT1G, Package_TO_SOT_SMD:SOT-23, F.Cu at (-17.2, 70.1)
- added R58: 33K, Resistor_SMD:R_0603_1608Metric_Pad0.98x0.95mm_HandSolder, F.Cu at (-95.1, 76.9)
- added R61: 33K, Resistor_SMD:R_0603_1608Metric_Pad0.98x0.95mm_HandSolder, F.Cu at (-95.1, 84.4)
- added R62: 33K, Resistor_SMD:R_0603_1608Metric_Pad0.98x0.95mm_HandSolder, F.Cu at (-95.1, 86.9)
- added R63: 33K, Resistor_SMD:R_0603_1608Metric_Pad0.98x0.95mm_HandSolder, F.Cu at (-95.1, 89.4)
- added R64: 1K, Resistor_SMD:R_0603_1608Metric_Pad0.98x0.95mm_HandSolder, F.Cu at (-90.8, 61.8)
- added R65: 2K2, Resistor_SMD:R_0603_1608Metric_Pad0.98x0.95mm_HandSolder, F.Cu at (-90.8, 64.3)
- added R66: 10R, MET:RES_10R_SMW210R, F.Cu at (-83.3, 81.0)
- added R67: 10K, Resistor_SMD:R_0603_1608Metric_Pad0.98x0.95mm_HandSolder, F.Cu at (-90.8, 66.8)
- added R68: 120R, Resistor_SMD:R_0603_1608Metric_Pad0.98x0.95mm_HandSolder, F.Cu at (-90.8, 69.3)
- added R69: 120R, Resistor_SMD:R_0603_1608Metric_Pad0.98x0.95mm_HandSolder, F.Cu at (-90.8, 71.8)
- added R70: 120R, Resistor_SMD:R_0603_1608Metric_Pad0.98x0.95mm_HandSolder, F.Cu at (-90.8, 74.4)
- added R71: 120R, Resistor_SMD:R_0603_1608Metric_Pad0.98x0.95mm_HandSolder, F.Cu at (-90.8, 76.9)
- added R72: 1K, Resistor_SMD:R_0805_2012Metric_Pad1.20x1.40mm_HandSolder, F.Cu at (-16.2, 7.83)
- added R73: 33R, Resistor_SMD:R_0805_2012Metric_Pad1.20x1.40mm_HandSolder, F.Cu at (-16.2, 10.8)
- added R74: 120R, Resistor_SMD:R_0603_1608Metric_Pad0.98x0.95mm_HandSolder, F.Cu at (-90.8, 79.4)
- added R75: 4K7, Resistor_SMD:R_0805_2012Metric_Pad1.20x1.40mm_HandSolder, F.Cu at (-16.2, 13.7)
- added R76: 0R, MET:RES_10R_SMW210R, F.Cu at (-83.3, 86.8)
- added TP15: 5002, MET:TP_5001, F.Cu at (-47.3, 110.0)
- added TP16: 5001, MET:TP_5001, F.Cu at (-47.3, 113.8)
- added TP17: 5002, MET:TP_5001, F.Cu at (-47.3, 117.5)
- added U4: TME-0505S, MET:TME-0505S, F.Cu at (-41.2, 122.6)
- moved D10 227.5 mm to (-81.5, 105.2)
- moved D11 227.5 mm to (-81.5, 113.0)
- moved D7 224.7 mm to (-93.6, 109.1)
- moved D8 224.7 mm to (-93.6, 112.2)
- moved D4 224.6 mm to (-98.1, 112.2)
- moved U2 221.3 mm to (-107.5, 97.8)
- moved J2 221.3 mm to (-94.5, 97.3)
- moved D9 221.2 mm to (-89.1, 102.9)
- moved D5 220.9 mm to (-93.6, 102.9)
- moved D6 220.9 mm to (-93.6, 106.0)
- moved IC6 217.8 mm to (-104.3, 119.3)
- moved D12 202.7 mm to (-80.9, 92.9)
- moved D13 202.7 mm to (-80.9, 97.5)
- moved TP12 192.6 mm to (-51.0, 113.8)
- moved TP13 192.6 mm to (-51.0, 117.5)
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Connections:
- C44 pad 2: /FilamentControl/MONITOR_IFIL -> MONITOR_IFIL
- C50 pad 1: /Monitor/uC_VFIL_ANL -> uC_VFIL_ANL
- C51 pad 1: /Monitor/uC_TAMP_ANL -> uC_TAMP_ANL
- D12 pad 2: /FilamentControl/MONITOR_IFIL -> MONITOR_IFIL
- D13 pad 2: /FilamentControl/MONITOR_IFIL -> MONITOR_IFIL
- D14 pad 2: /Monitor/FILOUT -> FILOUT
- D15 pad 2: /Monitor/uC_VFIL_ANL -> uC_VFIL_ANL
- D16 pad 2: /Monitor/MONITOR_24VNEG -> MONITOR_24VNEG
- D17 pad 2: /Monitor/uC_24VNEG_ANL -> uC_24VNEG_ANL
- D19 pad 2: /Monitor/uC_24V_ANL -> uC_24V_ANL
- D20 pad 2: /Monitor/uC_IFIL_ANL -> uC_IFIL_ANL
- D21 pad 1: /Monitor/uC_IFIL_ANL -> uC_IFIL_ANL
- D22 pad 2: /Monitor/FILOUT -> FILOUT
- D23 pad 2: /Monitor/uC_TAMP_ANL -> uC_TAMP_ANL
- D24 pad 2: /Monitor/uC_IFREQ_ANL -> uC_IFREQ_ANL
- IC5 pad 7: /FilamentControl/MONITOR_24VNEG -> MONITOR_24VNEG
- IC6 pad 2: /FilamentControl/uC_CS -> uC_CS
- IC6 pad 3: /FilamentControl/uC_CLK -> uC_CLK
- IC6 pad 4: /FilamentControl/uC_SDO -> uC_SDO
- J1 pad 1: /POWER/+B1 -> /POWER/-B1
- J1 pad 2: /POWER/-B1 -> /POWER/+B2
- J1 pad 3: /POWER/+B2 -> /POWER/+B1
- Q7 pad 1: /FilamentControl/uC_REFDIS -> uC_REFDIS
- R29 pad 2: /FilamentControl/MONITOR_TAMP -> MONITOR_TAMP
- R30 pad 1: /FilamentControl/FILOUT -> FILOUT
- R31 pad 1: /FilamentControl/FILOUT -> FILOUT
- R32 pad 1: /FilamentControl/MONITOR_IFIL -> MONITOR_IFIL
- R33 pad 1: /FilamentControl/MONITOR_IFIL -> MONITOR_IFIL
- R34 pad 2: /FilamentControl/MONITOR_IFIL -> MONITOR_IFIL
- R36 pad 1: /FilamentControl/MONITOR_24VNEG -> MONITOR_24VNEG
- R43 pad 1: /FilamentControl/MONITOR_IFIL -> MONITOR_IFIL
- R47 pad 1: /FilamentControl/uC_REFDIS -> uC_REFDIS
- R48 pad 1: /Monitor/uC_VFIL_ANL -> uC_VFIL_ANL
- R49 pad 2: /Monitor/uC_VFIL_ANL -> uC_VFIL_ANL
- R51 pad 1: /Monitor/uC_24VNEG_ANL -> uC_24VNEG_ANL
- R52 pad 2: /Monitor/uC_24V_ANL -> uC_24V_ANL
- R53 pad 1: /Monitor/uC_24V_ANL -> uC_24V_ANL
- R54 pad 1: /Monitor/uC_IFIL_ANL -> uC_IFIL_ANL
- R54 pad 2: /Monitor/MONITOR_IFIL -> MONITOR_IFIL
- R55 pad 2: /Monitor/uC_IFIL_ANL -> uC_IFIL_ANL
- R56 pad 1: /Monitor/uC_TAMP_ANL -> uC_TAMP_ANL
- R56 pad 2: /Monitor/MONITOR_TAMP -> MONITOR_TAMP
- R57 pad 2: /Monitor/uC_TAMP_ANL -> uC_TAMP_ANL
- R59 pad 1: /Monitor/uC_IFREQ_ANL -> uC_IFREQ_ANL
- R60 pad 2: /Monitor/uC_IFREQ_ANL -> uC_IFREQ_ANL
- T1 pad 2: /FilamentControl/FILOUT -> FILOUT
- TP13 pad 1: /FilamentControl/MONITOR_IFIL -> MONITOR_IFIL
- U2 pad 10: /uController/uC_24V_ANL -> uC_24V_ANL
- U2 pad 11: /uController/uC_24VNEG_ANL -> uC_24VNEG_ANL
- U2 pad 12: /uController/uC_TAMP_ANL -> uC_TAMP_ANL
- U2 pad 14: /uController/uC_IFREQ_ANL -> uC_IFREQ_ANL
- U2 pad 15: /uController/uC_IFREQ_ANL -> uC_IFREQ_ANL
- U2 pad 16: /uController/uC_EXT_OUT1 -> uC_EXT_OUT1
- U2 pad 17: /uController/uC_EXT_OUT2 -> uC_EXT_OUT2
- U2 pad 18: /uController/uC_EXT_IN1 -> uC_EXT_IN1
- U2 pad 19: /uController/uC_EXT_IN2 -> uC_EXT_IN2
- U2 pad 25: /uController/uC_SDO -> uC_SDO
- U2 pad 26: /uController/uC_CLK -> uC_CLK
- U2 pad 27: /uController/uC_CS -> uC_CS
- U2 pad 28: /uController/uC_REFDIS -> uC_REFDIS
- U2 pad 35: /uController/uC_FOCUS_AB -> uC_FOCUS_AB
- U2 pad 36: /uController/uC_FOCUS_A12 -> uC_FOCUS_A12
- U2 pad 37: /uController/uC_FOCUS_B12 -> uC_FOCUS_B12
- U2 pad 38: /uController/uC_FILON -> uC_FILON
- U2 pad 4: /uController/uC_IANODE_ANL -> uC_IANODE_ANL
- U2 pad 43: /uController/uC_CAN_TX0 -> uC_CAN_TX0
- U2 pad 44: /uController/uC_CAN_RX0 -> uC_CAN_RX0
- U2 pad 5: /uController/uC_IFIL_ANL -> uC_IFIL_ANL
- U2 pad 6: /uController/uC_VFIL_ANL -> uC_VFIL_ANL
- U3 pad 1: /FilamentControl/MONITOR_TAMP -> MONITOR_TAMP
Other:
- board outline added: 100 x 150 mm
