File: KiCad/PCB336/PCB336.kicad_pcb (KiCad board)
At the start: 2 copper layers, 100 x 150 mm, 244 parts, among them IC1 NJM78L12UA-TE1, IC10 ADM4857ARZ-REEL7, IC11 ADM4857ARZ-REEL7, IC12 MAX22246CAWA_V+, IC13 TJA1050T_CM,118, IC14 ESD2CAN24DBZRQ1, IC15 NJM78L05UA-TE1, IC2 NJM79L12SU3-TE1, IC3 TSR_0.5-2450, IC4 XR2206CP-F, IC5 LM1458MX_NOPB, IC6 MCP4821-E/MS, IC7 LM358BAIDR, IC8 ADUM3195BRQZ, IC9 ISO6742FDWR, J1 39-29-9043, J2 61200621621, J3 Piazzolato, J4 MOLEX_172298-1108, J5 105310-2210, J6 105310-2210, J7 105312-1104, J8 105312-1104, K1 32.21.7.024.4000, K2 32.21.7.024.4000, K3 32.21.7.024.4000, K4 32.21.7.024.4000, Q1 2N7002LT1G, Q10 2N7002LT1G, Q11 2N7002LT1G, Q2 2N7002LT1G, Q3 2N7002LT1G, Q4 2N7002LT1G, Q5 2N7002LT1G, Q6 2N7002LT1G, Q7 2N7002LT1G, Q8 2N7002LT1G, Q9 2N7002LT1G, T1 TF-108, U1 NCP1117ST33T3G, U2 ATSAME51J20A-A, U3 PCB319-2, U4 TME-0505S

Commit message: Iniziato loi sbroglio
Parts:
- removed C64: 1uF, Capacitor_SMD:C_1206_3216Metric_Pad1.33x1.80mm_HandSolder
- removed J6: 105310-2210, MET:1053102210
- removed TP10: 5002, MET:TP_5001
- added D32: GREEN, MET:LED_0805, F.Cu at (118.5, 45.0)
- added D33: GREEN, MET:LED_0805, F.Cu at (118.5, 49.5)
- added D34: GREEN, MET:LED_0805, F.Cu at (118.5, 36.0)
- added D35: YELLOW, MET:LED_0805, F.Cu at (126.0, 84.5)
- added D36: YELLOW, MET:LED_0805, F.Cu at (126.0, 86.8)
- added D37: YELLOW, MET:LED_0805, F.Cu at (126.0, 89.0)
- added R77: 2K2, Resistor_SMD:R_0805_2012Metric_Pad1.20x1.40mm_HandSolder, B.Cu at (118.5, 45.0)
- added R78: 2K2, Resistor_SMD:R_0805_2012Metric_Pad1.20x1.40mm_HandSolder, B.Cu at (118.5, 49.5)
- added R79: 680R, Resistor_SMD:R_0805_2012Metric_Pad1.20x1.40mm_HandSolder, B.Cu at (118.5, 36.0)
- added R81: 680R, Resistor_SMD:R_0603_1608Metric_Pad0.98x0.95mm_HandSolder, F.Cu at (122.2, 82.5)
- added R82: 680R, Resistor_SMD:R_0603_1608Metric_Pad0.98x0.95mm_HandSolder, F.Cu at (122.2, 84.2)
- added R83: 680R, Resistor_SMD:R_0603_1608Metric_Pad0.98x0.95mm_HandSolder, F.Cu at (122.4, 87.0)
- added R84: 680R, Resistor_SMD:R_0603_1608Metric_Pad0.98x0.95mm_HandSolder, F.Cu at (122.5, 88.8)
- C15, C27, C28, C30, C32, C34, C35, C36, C37, C38, C39, C44, C46, C47, C48, C49, C50, C52, C53, C54, C55, C56, C57, C58, C59, C60, C61, C62, D10, D11, D12, D13, D14, D15, D22, D24, D25, D26, D27, D28, IC10, IC11, IC5, IC7, IC8, IC9, Q1, Q10, Q11, Q2, Q3, Q4, Q5, Q6, Q7, Q8, Q9, R1, R11, R13, R15, R17, R19, R2, R20, R21, R22, R24, R25, R26, R27, R28, R29, R30, R31, R32, R33, R34, R35, R36, R38, R39, R40, R41, R42, R43, R44, R45, R46, R47, R48, R49, R58, R59, R60, R61, R62, R63, R64, R65, R67, R68, R69, R70, R71, R8, R9: moved to B.Cu
- D21: value 1N4148W -> YELLOW; footprint Diode_SMD:D_SOD-123 -> MET:LED_0805
- D29: value ESDM2032MX4T5G -> MMBZ6V2AL,215; footprint MET:ESDM2032MX4T5G -> MET:MMBZ6V2AL,215; moved to B.Cu
- R3: value 1K -> 870R; moved to B.Cu
- R76: footprint MET:RES_10R_SMW210R -> Resistor_SMD:R_0603_1608Metric_Pad0.98x0.95mm_HandSolder; moved to B.Cu
- moved K1 273.3 mm to (130.5, 135.5), turned to 180 degrees
- moved K3 270.7 mm to (130.7, 149.0), turned to 180 degrees
- moved R9 242.0 mm to (126.5, 41.5), turned to 90 degrees
- moved R13 241.4 mm to (126.5, 55.5), turned to 90 degrees
- moved R8 241.1 mm to (126.5, 45.0), turned to 90 degrees
- moved R11 240.4 mm to (126.5, 59.0), turned to 90 degrees
- moved K2 239.9 mm to (99.5, 134.8), turned to -90 degrees
- moved U3 239.6 mm to (93.0, 163.2), turned to 90 degrees
- moved R10 239.5 mm to (123.4, 41.0)
- moved K4 239.3 mm to (99.5, 158.0), turned to -90 degrees
- moved R7 238.0 mm to (123.6, 44.5)
- moved R12 237.9 mm to (123.7, 58.5)
- moved IC9 236.3 mm to (126.9, 87.8), turned to 90 degrees
- moved R17 235.6 mm to (126.5, 48.5), turned to 90 degrees
- moved D4 235.5 mm to (127.4, 44.5)
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Connections:
- C30 pad 1: GND -> GNDPWR
- C31 pad 1: GND -> GNDPWR
- C32 pad 1: GND -> GNDPWR
- C33 pad 1: GND -> GNDPWR
- C35 pad 1: GND -> GNDPWR
- C36 pad 1: GND -> GNDPWR
- C37 pad 1: GND -> GNDPWR
- C39 pad 1: GND -> GNDPWR
- C44 pad 1: GND -> GNDPWR
- C45 pad 2: GND -> GNDPWR
- C46 pad 2: GND -> GNDPWR
- C49 pad 1: GND -> GNDPWR
- C63 pad 1: GND_EXT -> +3V3
- C63 pad 2: +5V_EXT -> GNDPWR
- D12 pad 1: GND -> GNDPWR
- D13 pad 1: GND -> GNDPWR
- D21 pad 1: uC_IFIL_ANL -> GND_EXT
- D21 pad 2: GND -> Net-(D21-A)
- D29 pad 1: Earth -> GNDPWR
- D29 pad 2: GNDPWR -> Earth
- IC5 pad 5: GND -> GNDPWR
- IC6 pad 5: GND -> GNDPWR
- IC6 pad 7: GND -> GNDPWR
- IC7 pad 4: GND -> GNDPWR
- J1 pad 2: /POWER/+B2 -> /POWER/-B2
- J1 pad 4: /POWER/-B2 -> /POWER/+B2
- J3 pad 2: +12V -> /FilamentControl/fo
- J3 pad 3: GND -> +12V
- J3 pad 5: /FilamentControl/fo -> GNDPWR
- J4 pad 3: Earth -> GNDPWR
- J4 pad 8: GNDPWR -> Earth
- J5 pad 1: /ExternalSynch/EXT_OUT1+ -> /ExternalSynch/EXT_IN1-
- J5 pad 2: /ExternalSynch/EXT_OUT1- -> /ExternalSynch/EXT_IN1+
- J5 pad 3: /ExternalSynch/EXT_IN1+ -> +5V_EXT
- J5 pad 4: /ExternalSynch/EXT_IN1- -> /ExternalSynch/EXT_OUT2-
- J5 pad 5: GND_EXT -> /ExternalSynch/EXT_OUT2+
- J5 pad 6: +5V_EXT -> /ExternalSynch/EXT_OUT1-
- J5 pad 7: /ExternalSynch/EXT_OUT2+ -> /ExternalSynch/EXT_OUT1+
- J5 pad 8: /ExternalSynch/EXT_OUT2- -> GND_EXT
- Q7 pad 2: GND -> GNDPWR
- R20 pad 2: GND -> GNDPWR
- R24 pad 2: GND -> GNDPWR
- R25 pad 2: GND -> GNDPWR
- R28 pad 2: GND -> GNDPWR
- R32 pad 2: GND -> GNDPWR
- R33 pad 2: GND -> GNDPWR
- R39 pad 1: GND -> GNDPWR
- R41 pad 1: GND -> GNDPWR
- RV2 pad 3: GND -> GNDPWR
- U2 pad 24: /uController/LED4 -> unconnected-(U2-PB11-Pad24)
- U2 pad 39: /uController/LED3 -> /uController/LED_VTL
- U2 pad 40: /uController/LED2 -> /uController/LED_FLT
- U2 pad 41: unconnected-(U2-PA20-Pad41) -> /uController/LED4
- U2 pad 42: unconnected-(U2-PA21-Pad42) -> /uController/LED3
- U2 pad 45: unconnected-(U2-PA24-Pad45) -> /uController/LED2
- U2 pad 46: unconnected-(U2-PA25-Pad46) -> /uController/LED1
- U2 pad 49: /uController/LED1 -> unconnected-(U2-PB22-Pad49)
- U2 pad 50: /uController/LED_FLT -> unconnected-(U2-PB23-Pad50)
- U2 pad 60: /uController/LED_VTL -> unconnected-(U2-PB31-Pad60)
- U3 pad 2: GND -> GNDPWR
- U3 pad 6: -24V -> unconnected-(U3-nc2-Pad6)
Routing:
- net -24V: track 0.00 -> 257.9 mm, vias 0 -> 14
- net +24V: track 0.00 -> 237.8 mm, vias 0 -> 7
- net GNDPWR: track 0.00 -> 205.4 mm, vias 0 -> 13
- net GND: track 0.00 -> 106.7 mm
- net /POWER/+B2: track 0.00 -> 54.8 mm, vias 0 -> 4
- net /POWER/+B1: track 0.00 -> 36.9 mm, vias 0 -> 3
- net /POWER/-B2: track 0.00 -> 28.4 mm, vias 0 -> 3
- net /POWER/-B1: track 0.00 -> 21.2 mm, vias 0 -> 2
- net Net-(FL1-INPUT): track 0.00 -> 19.7 mm, vias 0 -> 3
- net +3V3: track 0.00 -> 18.7 mm
- net Net-(FL2-INPUT): track 0.00 -> 18.6 mm, vias 0 -> 2
- net Net-(C13-+): track 0.00 -> 17.6 mm
- net +5V: track 0.00 -> 11.9 mm
- net +12V: track 0.00 -> 5.16 mm
- added copper zone on B.Cu, net GNDPWR
- added copper zone on F.Cu, net GNDPWR
- added copper zone on In1.Cu, net GNDPWR
- added copper zone on In2.Cu, net GNDPWR
Other:
- outline, holes or cut-outs redrawn
- copper layers 2 -> 4
- board text added: "+12V"
- board text added: "+24V"
- board text added: "+3V3"
- board text added: "+5V"
- board text added: "-12V"
- board text added: "-24V"
- board text added: "FAB"
- board text added: "FEN"
- board text added: "FGP"
- board text added: "FLT"
- board text added: "FON"
- board text added: "GND"
- board text added: "GNDP"
- board text added: "IANODE"
- board text added: "ICAL"
- board text added: "IFIL"
- board text added: "IN1"
- board text added: "IN2"
- board text added: "ISYM"
- board text added: "OUT1"
- board text added: "OUT2"
- board text added: "VFIL"
- board text added: "VREF"
- board text added: "VTL"
