File: KiCad/PCB336/filamentcontrol.kicad_sch (KiCad schematic)
At the start: 36 parts, among them IC4 XR2206CP-F, IC5 LM1458MX_NOPB, T1 TF-108, U3 PCB319-2

Commit message: Completato Filament e Monitor
Parts:
- added C44: 10uF, Capacitor_SMD:C_1206_3216Metric_Pad1.33x1.80mm_HandSolder, symbol Device:C_Small
- added C45, C46, C47: 100nF, Capacitor_SMD:C_0805_2012Metric_Pad1.18x1.45mm_HandSolder, symbol Device:C_Small
- added C48: 47nF, Capacitor_SMD:C_0805_2012Metric_Pad1.18x1.45mm_HandSolder, symbol Device:C_Small
- added C49: 1uF, Capacitor_SMD:C_1206_3216Metric_Pad1.33x1.80mm_HandSolder, symbol Device:C_Small
- added D12, D13: BAT754S,215, MET:BAT754S,215, symbol MET:BAT754S,215
- added IC6: MCP4821-E/MS, MET:MCP4821_EMS, symbol MET:MCP4821-E_MS
- added IC7: LM358BAIDR, MET:LM358BAIDR, symbol MET:LM358BAIDR
- added J3: Piazzolato, Connector_PinSocket_2.54mm:PinSocket_1x05_P2.54mm_Vertical, symbol Connector_Generic:Conn_01x05
- added Q7: 2N7002LT1G, Package_TO_SOT_SMD:SOT-23, symbol Transistor_FET:2N7002
- added R30, R31: 4K7, Resistor_SMD:R_1206_3216Metric_Pad1.30x1.75mm_HandSolder, symbol Device:R
- added R32, R33: 200R, Resistor_SMD:R_0603_1608Metric_Pad0.98x0.95mm_HandSolder, symbol Device:R
- added R34, R36, R37, R38, R39, R42, R43: 10K, Resistor_SMD:R_0603_1608Metric_Pad0.98x0.95mm_HandSolder, symbol Device:R
- added R35: 87K, Resistor_SMD:R_0603_1608Metric_Pad0.98x0.95mm_HandSolder, symbol Device:R
- added R40: 39K, Resistor_SMD:R_0603_1608Metric_Pad0.98x0.95mm_HandSolder, symbol Device:R
- added R41: 27K, Resistor_SMD:R_0603_1608Metric_Pad0.98x0.95mm_HandSolder, symbol Device:R
- added R44, R47: 4K7, Resistor_SMD:R_0603_1608Metric_Pad0.98x0.95mm_HandSolder, symbol Device:R
- added R45: 5K6, Resistor_SMD:R_0603_1608Metric_Pad0.98x0.95mm_HandSolder, symbol Device:R
- added R46: 18K, Resistor_SMD:R_0603_1608Metric_Pad0.98x0.95mm_HandSolder, symbol Device:R
- added RV2: 5K, Potentiometer_THT:Potentiometer_Bourns_3296W_Vertical, symbol Device:R_Potentiometer
- added TP11, TP13, TP14: 5002, MET:TP_5001, symbol MET:TP_Serie_5001
- added TP12: 5001, MET:TP_5001, symbol MET:TP_Serie_5001
Connections:
- net +12V: now also C49.2, IC7.8 (V+), J3.2 (Pin_2)
- net +5V: now also R34.1
- net -12V: now also J3.4 (Pin_4)
- net -24V: now also R35.2
- net GND: now also IC5.5 (+B), C44.1, C45.2, C46.2, C49.1, D12.1 (A), D13.1 (A), IC6.5 (~{LDAC}), IC6.7 (VSS), IC7.4 (V-), J3.3 (Pin_3), Q7.2 (S), R32.2, R33.2, R39.1, R41.1, RV2.3
- net GNDPWR: now also R30.2, R31.2, TP12.1
- net ffdb: now also J3.1 (Pin_1), R46.2
- net fo: now also J3.5 (Pin_5)
- net at C43.2, D11.2 (A), T1.1 (P1): now also TP11.1
- net FILOUT: now reaches T1.2 (P2)
- net FILOUT: now also R30.1, R31.1
- net VFA: now reaches T1.3 (O1)
- net VFA: now also D12.3 (COM)
- net VFB: now reaches T1.4 (O2)
- net VFB: now also D13.3 (COM)
- net at IC5.6 (-B): now also R35.1, R36.2
- net MONITOR_24VNEG: now reaches IC5.7 (OB)
- net MONITOR_24VNEG: now also R36.1
- net uC_Tamp renamed MONITOR_TAMP
- new net: IC7.2 (IN1-), R38.2, R39.2
- new net: IC6.6 (~{SHDN}), R37.1
- new net: IC6.8 (VOUT), IC7.3 (IN1+)
- new net: IC7.1 (OUT1), R38.1, R40.2
- new net: C47.2, R42.1, R43.2
- new net: C47.1, C48.2, IC7.6 (IN2-), R42.2, R44.2
- new net: C48.1, R45.1
- new net: IC7.7 (OUT2), R45.2, R46.1
- new net: R44.1, RV2.1, RV2.2
- new net +3V3: C45.1, IC6.1 (VDD), R37.2, R47.2
- new net MONITOR_IFIL: C44.2, D12.2 (K), D13.2 (K), R32.1, R33.1, R34.2, R43.1, TP13.1
- new net uC_CLK: IC6.3 (SCK)
- new net uC_CS: IC6.2 (~{CS})
- new net uC_REFDIS: Q7.1 (G), R47.1
- new net uC_SDO: IC6.4 (SDI)
- new net vref: C46.1, IC7.5 (IN2+), Q7.3 (D), R40.1, R41.2, TP14.1
Other:
- note added: "ABILITAZIONE FILAMENTO"
- note added: "DAC OUTPUT 2.048V MAX"
- note added: "Error Amplifier"
- note added: "INPUT SIGNAL"
- note added: "MONITOR -24V POWER SUPPLY"
- note added: "MONITOR TEMP. AMPLI"
- note added: "PRE-AMPLI FEEDBACK"
- note added: "Predisposizione Sostituzione XR2206"
- note added: "REGOLAZIONE LIVELLO DI RIFERIMENTO"
- note added: "Regolazione Simmetria Uscita"
- note added: "VCO Error Feedback"
- note added: "VFEED = Irms * 0.9"
- note added: "Valore Medio Corrente di filamento"
- note added: "Vref = 2.048 * 0.818"
- moved on the sheet: C28, C34, C35, C36, C37, C38, C39, IC5, R24, R25, R26, R27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

Commit message: Completato schematico, e ERC Iniziato piazzamento
Other:
- moved on the sheet: C28, C34, C35, C36, C37, C38, IC5, R24, R25, R26, R27, R28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

Commit message: Iniziato loi sbroglio
Parts:
- removed TP10: 5002, MET:TP_5001, symbol MET:TP_Serie_5001
- added C3, C6: 33uF, MET:WCAP-HTG5_D8_H9_P3.5, symbol MET:WCAP-HTG5
- added C63: 1uF, Capacitor_SMD:C_1206_3216Metric_Pad1.33x1.80mm_HandSolder, symbol Device:C_Small
Connections:
- net +12V: now also J3.3 (Pin_3); no longer J3.2 (Pin_2)
- net +24V: now also C3.1
- net +3V3: now also C63.1
- net -24V: now also C6.2; no longer U3.6 (nc2)
- net GNDPWR: now also C30.1, C31.1, C32.1, C33.1, C35.1, C36.1, C37.1, C39.1, C44.1, C45.2, C46.2, C49.1, D12.1 (A), D13.1 (A), IC5.5 (+B), IC6.5 (~{LDAC}), IC6.7 (VSS), IC7.4 (V-), J3.5 (Pin_5), Q7.2 (S), R20.2, R24.2, R25.2, R28.2, R32.2, R33.2, R39.1, R41.1, RV2.3, U3.2 (-T), C3.2, C6.1, C63.2
- net fo: now also J3.2 (Pin_2); no longer J3.5 (Pin_5)
- removed net GND: C30.1, C31.1, C32.1, C33.1, C35.1, C36.1, C37.1, C39.1, C44.1, C45.2, C46.2, C49.1, D12.1 (A), D13.1 (A), IC5.5 (+B), IC6.5 (~{LDAC}), IC6.7 (VSS), IC7.4 (V-), J3.3 (Pin_3), Q7.2 (S), R20.2, R24.2, R25.2, R28.2, R32.2, R33.2, R39.1, R41.1, RV2.3, U3.2 (-T)
