File: KiCad/PCB336/power.kicad_sch (KiCad schematic)
At the start: 41 parts, among them IC1 NJM78L12UA-TE1, IC2 NJM79L12SU3-TE1, IC3 TSR_0.5-2450, J1 39-29-9043, U1 NCP1117ST33T3G

Commit message: Filament Pagina in lavorazione
Parts:
- removed TP2: RED, MET:TP_5001, symbol MET:TP_Serie_5001
- added TP9: 5000, MET:TP_5001, symbol MET:TP_Serie_5001
- D1, D2, D3: Color (none) -> GREEN
- TP1, TP4, TP5, TP6, TP7: value RED -> 5000; Color (none) -> RED
- TP3: value BLACK -> 5001; Color (none) -> BLACK
Connections:
- net -24V: now also TP9.1
Other:
- company: (none) -> METALTRONICA
- title: (none) -> PCB/25-336-1

Commit message: Avanzamenti in Agosto
Connections:
- net GND1 renamed GNDPWR
Changed lines of the file:
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@@
-	)
-	(symbol
-		(lib_id "power:GND1")
-		(at 115.57 55.88 0)
-		(unit 1)
-		(body_style 1)
-		(exclude_from_sim no)
-		(in_bom yes)
-		(on_board yes)
-		(in_pos_files yes)
-		(dnp no)
-		(fields_autoplaced yes)
-		(property "Reference" "#PWR02"
-			(at 115.57 62.23 0)
-			(hide yes)
-			(show_name no)
-			(do_not_autoplace no)
-			(effects
-				(font
-					(size 1.27 1.27)
-				)
-			)
-		)
-		(property "Value" "GND1"
-			(at 115.57 60.96 0)
-			(show_name no)
-			(do_not_autoplace no)
-			(effects
-				(font
-					(size 1.27 1.27)
-				)
-			)
-		)
-		(property "Footprint" ""
-			(at 115.57 55.88 0)
-			(hide yes)
-			(show_name no)
-			(do_not_autoplace no)
-			(effects
-				(font
-					(size 1.27 1.27)
-				)
-			)
-		)
-		(property "Datasheet" ""
-			(at 115.57 55.88 0)
-			(hide yes)
-			(show_name no)
-			(do_not_autoplace no)
-			(effects
-				(font
-					(size 1.27 1.27)
-				)
-			)
-		)
-		(property "Description" "Power symbol creates a global label with name \"GND1\" , ground"
-			(at 115.57 55.88 0)
-			(hide yes)
-			(show_name no)
-			(do_not_autoplace no)
-			(effects
-				(font
-					(size 1.27 1.27)
-				)
-			)
-		)
-		(pin "1"
-		)
-		(instances
-			(project "PCB336"
-				(path "/f1a2d35c-afab-4479-8747-9ab1a9f252d1"
-					(reference "#PWR02")
-					(unit 1)
-				)
-			)
-		)
 	)
 	(symbol
@@
 					(unit 1)
 				)
+			)
+		)
+	)
+	(symbol
+		(lib_id "power:GNDPWR")
+		(at 115.57 55.88 0)
+		(unit 1)
+		(body_style 1)
+		(exclude_from_sim no)
+		(in_bom yes)
+		(on_board yes)
+		(in_pos_files yes)
+		(dnp no)
+		(fields_autoplaced yes)
+		(property "Reference" "#PWR02"
+			(at 115.57 60.96 0)
+			(hide yes)
+			(show_name no)
+			(do_not_autoplace no)
+			(effects
+				(font
+					(size 1.27 1.27)
+				)
+			)
+		)
+		(property "Value" "GNDPWR"
+			(at 115.443 59.69 0)
+			(show_name no)
+			(do_not_autoplace no)
+			(effects
+				(font
+					(size 1.27 1.27)
+				)
+			)
+		)
+		(property "Footprint" ""
+			(at 115.57 57.15 0)
+			(hide yes)
+			(show_name no)
+			(do_not_autoplace no)
+			(effects
+				(font
+					(size 1.27 1.27)
+				)
+			)
+		)
+		(property "Datasheet" ""
+			(at 115.57 57.15 0)
+			(hide yes)
+			(show_name no)
+			(do_not_autoplace no)
+			(effects
+				(font
+					(size 1.27 1.27)
+				)
+			)
+		)
+		(property "Description" "Power symbol creates a global label with name \"GNDPWR\" , global ground"
+			(at 115.57 55.88 0)
+			(hide yes)
+			(show_name no)
+			(do_not_autoplace no)
+			(effects
+				(font
+					(size 1.27 1.27)
+				)
+			)
+		)
+		(pin "1"
+		)
+		(instances
+			(project "PCB336"
+				(path "/f1a2d35c-afab-4479-8747-9ab1a9f252d1"
+					(reference "#PWR02")
+					(unit 1)
+				)

Commit message: Completato Filament e Monitor
Parts:
- JP1: footprint (none) -> Jumper:SolderJumper-2_P1.3mm_Bridged2Bar_Pad1.0x1.5mm
Changed lines of the file:
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@@
 	(title_block
 		(title "PCB/25-336-1")
+		(date "2026-09-01")
 		(rev "0")
 		(company "METALTRONICA")
@@
 			)
 		)
-		(property "Footprint" ""
+		(property "Footprint" "Jumper:SolderJumper-2_P1.3mm_Bridged2Bar_Pad1.0x1.5mm"
 			(at 153.67 59.69 0)
 			(hide yes)

Commit message: Completato schematico, e ERC Iniziato piazzamento
Connections:
- net +B1: now also J1.3 (Pin_3); no longer J1.1 (Pin_1)
- net +B2: now also J1.2 (Pin_2); no longer J1.3 (Pin_3)
- net -B1: now also J1.1 (Pin_1); no longer J1.2 (Pin_2)

Commit message: Iniziato loi sbroglio
Parts:
- removed C3, C6: 33uF, MET:WCAP-HTG5_D8_H9_P3.5, symbol MET:WCAP-HTG5
- added D32, D33, D34: GREEN, MET:LED_0805, symbol Device:LED
- added R77, R78: 2K2, Resistor_SMD:R_0805_2012Metric_Pad1.20x1.40mm_HandSolder, symbol Device:R
- added R79: 680R, Resistor_SMD:R_0805_2012Metric_Pad1.20x1.40mm_HandSolder, symbol Device:R
- R3: value 1K -> 870R
Connections:
- net +12V: now also D32.2 (A)
- net +3V3: now also D34.2 (A)
- net +B2: now also J1.4 (Pin_4); no longer J1.2 (Pin_2)
- net -12V: now also D33.1 (K)
- net -B2: now also J1.2 (Pin_2); no longer J1.4 (Pin_4)
- net GND: now also R77.2, R78.2, R79.2
- new net: D34.1 (K), R79.1
- new net: D32.1 (K), R77.1
- new net: D33.2 (A), R78.1
