File: KiCad/PCB336/ucontroller.kicad_sch (KiCad schematic)
At the start: 17 parts, among them J2 61200621621, U2 ATSAME51J20A-A

Commit message: Filament Pagina in lavorazione
Parts:
- added D4: BLUE, MET:LED_0805, symbol Device:LED
- added D5: RED, MET:LED_0805, symbol Device:LED
- added D6, D7, D8, D9: YELLOW, MET:LED_0805, symbol Device:LED
- added Q1, Q2, Q3, Q4, Q5, Q6: 2N7002LT1G, Package_TO_SOT_SMD:SOT-23, symbol Transistor_FET:2N7002
- added R10, R12, R14, R16, R18, R7: 680R, Resistor_SMD:R_0603_1608Metric_Pad0.98x0.95mm_HandSolder, symbol Device:R
- added R11, R13, R15, R17, R8, R9: 33K, Resistor_SMD:R_0603_1608Metric_Pad0.98x0.95mm_HandSolder, symbol Device:R
Connections:
- net GND: now also Q1.2 (S), Q2.2 (S), Q3.2 (S), Q4.2 (S), Q5.2 (S), Q6.2 (S), R11.2, R13.2, R15.2, R17.2, R8.2, R9.2
- net uC_24V_ANL: now reaches U2.10 (PB07)
- net uC_24VNEG_ANL: now reaches U2.11 (PB08)
- net uC_TAMP_ANL: now reaches U2.12 (PB09)
- net uC_FILFREQ: now reaches U2.14 (PA05)
- net uC_FILFREQ: now also U2.15 (PA06)
- net uC_EXT_OUT1: now reaches U2.16 (PA07)
- net uC_EXT_OUT2: now reaches U2.17 (PA08)
- net uC_EXT_IN1: now reaches U2.18 (PA09)
- net uC_EXT_IN2: now reaches U2.19 (PA10)
- net LED4: now reaches U2.24 (PB11)
- net LED4: now also Q6.1 (G), R17.1
- net uC_FOCUS_AB: now reaches U2.35 (PA16)
- net uC_FOCUS_A12: now reaches U2.36 (PA17)
- net uC_FOCUS_B12: now reaches U2.37 (PA18)
- net uC_FILON: now reaches U2.38 (PA19)
- net LED3: now reaches U2.39 (PB16)
- net LED3: now also Q5.1 (G), R15.1
- net uC_IANODE_ANL: now reaches U2.4 (PA03)
- net LED2: now reaches U2.40 (PB17)
- net LED2: now also Q4.1 (G), R13.1
- net LED1: now reaches U2.49 (PB22)
- net LED1: now also Q3.1 (G), R11.1
- net uC_IFIL_ANL: now reaches U2.5 (PB04)
- net LED_FLT: now reaches U2.50 (PB23)
- net LED_FLT: now also Q2.1 (G), R9.1
- net uC_VFILx5_ANL: now reaches U2.6 (PB05)
- net LED_VTL: now reaches U2.60 (PB31)
- net LED_VTL: now also Q1.1 (G), R8.1
- net uC_VFILx15_ANL: now reaches U2.9 (PB06)
- new net: D9.1 (K), Q6.3 (D)
- new net: D9.2 (A), R18.2
- new net: D4.1 (K), Q1.3 (D)
- new net: D4.2 (A), R7.2
- new net: D8.2 (A), R16.2
- new net: D6.1 (K), Q3.3 (D)
- new net: D6.2 (A), R12.2
- new net: D5.1 (K), Q2.3 (D)
- new net: D7.1 (K), Q4.3 (D)
- new net: D7.2 (A), R14.2
- new net: D8.1 (K), Q5.3 (D)
- new net: D5.2 (A), R10.2
- new net +5V: R10.1, R12.1, R14.1, R16.1, R18.1, R7.1
Other:
- company: (none) -> METALTRONICA
- title: (none) -> PCB/25-336-1

Commit message: Completato Filament e Monitor
Connections:
- net uC_FILFREQ renamed uC_IFREQ_ANL
- net uC_VFILx15_ANL: no longer names the net of U2.9 (PB06)
- net uC_VFILx5_ANL renamed uC_VFIL_ANL
Changed lines of the file:
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@@
 	(title_block
 		(title "PCB/25-336-1")
+		(date "2026-09-01")
 		(rev "0")
 		(company "METALTRONICA")
@@
 	)
 	(junction
-		(at 101.6 77.47)
-		(diameter 0)
-		(color 0 0 0 0)
-	)
-	(junction
 		(at 114.3 20.32)
 		(diameter 0)
@@
 	(junction
 		(at 137.16 36.83)
+		(diameter 0)
+		(color 0 0 0 0)
+	)
+	(junction
+		(at 101.6 76.2)
 		(diameter 0)
 		(color 0 0 0 0)
@@
 	(wire
 		(pts
-			(xy 101.6 76.2) (xy 101.6 77.47)
-		)
-		(stroke
-			(width 0)
-			(type default)
-		)
-	)
-	(wire
-		(pts
 			(xy 248.92 93.98) (xy 248.92 95.25)
 		)
@@
 	(wire
 		(pts
-			(xy 151.13 78.74) (xy 160.02 78.74)
-		)
-		(stroke
-			(width 0)
-			(type default)
-		)
-	)
-	(wire
-		(pts
 			(xy 151.13 96.52) (xy 161.29 96.52)
 		)
@@
 	(wire
 		(pts
-			(xy 95.25 77.47) (xy 101.6 77.47)
-		)
-		(stroke
-			(width 0)
-			(type default)
-		)
-	)
-	(wire
-		(pts
 			(xy 208.28 142.24) (xy 208.28 143.51)
 		)
@@
 	(wire
 		(pts
-			(xy 101.6 77.47) (xy 101.6 78.74)
+			(xy 101.6 76.2) (xy 101.6 78.74)
 		)
 		(stroke
@@
 		(pts
 			(xy 218.44 31.75) (xy 218.44 33.02)
+		)
+		(stroke
+			(width 0)
+			(type default)
+		)
+	)
+	(wire
+		(pts
+			(xy 93.98 76.2) (xy 101.6 76.2)
 		)
 		(stroke
@@
 		)
 	)
-	(label "uC_FILFREQ"
-		(at 95.25 77.47 180)
-		(effects
-			(font
-				(size 1.27 1.27)
-			)
-			(justify right bottom)
-		)
-	)
 	(label "Vuc"
 		(at 102.87 158.75 0)
@@
 		)
 	)
+	(label "uC_IFREQ_ANL"
+		(at 93.98 76.2 180)
+		(effects
+			(font
+				(size 1.27 1.27)
+			)
+			(justify right bottom)
+		)
+	)
 	(label "SVO"
 		(at 63.5 175.26 0)
@@
 		)
 	)
-	(label "uC_VFILx5_ANL"
+	(label "uC_VFIL_ANL"
 		(at 160.02 76.2 0)
 		(effects
@@
 		(effects
 			(font
-				(size 1.27 1.27)
-			)
-			(justify left bottom)
-		)
-	)
-	(label "uC_VFILx15_ANL"
-		(at 160.02 78.74 0)
-		(effects
-			(font

Commit message: Completato schematico, e ERC Iniziato piazzamento
Connections:
- no-connect marks 1 -> 21

Commit message: Iniziato loi sbroglio
Connections:
- net LED1: now also U2.46 (PA25); no longer U2.49 (PB22)
- net LED2: now also U2.45 (PA24); no longer U2.40 (PB17)
- net LED3: now also U2.42 (PA21); no longer U2.39 (PB16)
- net LED4: now also U2.41 (PA20); no longer U2.24 (PB11)
- net LED_FLT: now also U2.40 (PB17); no longer U2.50 (PB23)
- net LED_VTL: now also U2.39 (PB16); no longer U2.60 (PB31)
- no-connect marks 21 -> 17
Changed lines of the file:
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@@
-	)
-	(no_connect
-		(at 105.41 127)
 	)
 	(no_connect
@@
 	)
 	(no_connect
-		(at 105.41 116.84)
-	)
-	(no_connect
-		(at 105.41 114.3)
-	)
-	(no_connect
 		(at 105.41 66.04)
 	)
@@
 	)
 	(no_connect
-		(at 105.41 124.46)
-	)
-	(no_connect
 		(at 105.41 68.58)
 	)
@@
 	(wire
 		(pts
-			(xy 87.63 121.92) (xy 105.41 121.92)
+			(xy 67.31 121.92) (xy 105.41 121.92)
 		)
 		(stroke
@@
 	(wire
 		(pts
+			(xy 72.39 127) (xy 105.41 127)
+		)
+		(stroke
+			(width 0)
+			(type default)
+		)
+	)
+	(wire
+		(pts
 			(xy 125.73 46.99) (xy 125.73 41.91)
 		)
@@
 	(wire
 		(pts
+			(xy 72.39 124.46) (xy 105.41 124.46)
+		)
+		(stroke
+			(width 0)
+			(type default)
+		)
+	)
+	(wire
+		(pts
 			(xy 127 148.59) (xy 127 151.13)
 		)
@@
 	(wire
 		(pts
-			(xy 87.63 119.38) (xy 105.41 119.38)
+			(xy 67.31 119.38) (xy 105.41 119.38)
 		)
 		(stroke
@@
 	(wire
 		(pts
+			(xy 72.39 114.3) (xy 105.41 114.3)
+		)
+		(stroke
+			(width 0)
+			(type default)
+		)
+	)
+	(wire
+		(pts
 			(xy 218.44 52.07) (xy 218.44 57.15)
 		)
@@
 	(wire
 		(pts
+			(xy 72.39 116.84) (xy 105.41 116.84)
+		)
+		(stroke
+			(width 0)
+			(type default)
+		)
+	)
+	(wire
+		(pts
 			(xy 125.73 36.83) (xy 125.73 31.75)
 		)
@@
 			(width 0)
 			(type default)
-		)
-	)
-	(label "LED1"
-		(at 177.8 109.22 0)
-		(effects
-			(font
-				(size 1.27 1.27)
-			)
-			(justify left bottom)
 		)
 	)
@@
 	)
 	(label "LED2"
+		(at 72.39 124.46 0)
+		(effects
+			(font
+				(size 1.27 1.27)
+			)
+			(justify left bottom)
+		)
+	)
+	(label "LED2"
 		(at 246.38 93.98 180)
 		(effects
@@
 			)
 			(justify right bottom)
+		)
+	)
+	(label "LED_FLT"
+		(at 177.8 106.68 0)
+		(effects
+			(font
+				(size 1.27 1.27)
+			)
+			(justify left bottom)
 		)
 	)
@@
 		)
 	)
+	(label "LED4"
+		(at 72.39 114.3 0)
+		(effects
+			(font
+				(size 1.27 1.27)
+			)
+			(justify left bottom)
+		)
+	)
 	(label "Vuc"
 		(at 102.87 158.75 0)
@@
 		)
 	)
-	(label "LED_VTL"
-		(at 177.8 116.84 0)
-		(effects
-			(font
-				(size 1.27 1.27)
-			)
-			(justify left bottom)
-		)
-	)
 	(label "SWCLK"
 		(at 20.32 177.8 0)
@@
 		)
 	)
-	(label "LED_FLT"
-		(at 177.8 111.76 0)
-		(effects
-			(font
-				(size 1.27 1.27)
-			)
-			(justify left bottom)
-		)
-	)
 	(label "SWCLK"
 		(at 95.25 132.08 0)
@@
 		)
 	)
-	(label "LED4"
-		(at 177.8 91.44 0)
-		(effects
-			(font
-				(size 1.27 1.27)
-			)
-			(justify left bottom)
-		)
-	)
-	(label "LED3"
-		(at 177.8 104.14 0)
-		(effects
-			(font
-				(size 1.27 1.27)
-			)
-			(justify left bottom)
-		)
-	)
 	(label "MCLR"
 		(at 27.94 172.72 0)
@@
 		)
 	)
-	(label "LED2"
-		(at 177.8 106.68 0)
+	(label "LED1"
+		(at 72.39 127 0)
+		(effects
+			(font
+				(size 1.27 1.27)
+			)
+			(justify left bottom)
+		)
+	)
+	(label "LED_VTL"
+		(at 177.8 104.14 0)
 		(effects
 			(font
@@
 			)
 			(justify right bottom)
+		)
+	)
+	(label "LED3"
+		(at 72.39 116.84 0)
+		(effects
+			(font
+				(size 1.27 1.27)
+			)
+			(justify left bottom)
 		)
 	)
@@
 	(global_label "uC_CAN_RX0"
 		(shape input)
-		(at 87.63 121.92 180)
+		(at 67.31 121.92 180)
 		(fields_autoplaced yes)
 		(effects
@@
 		)
 		(property "Intersheetrefs" "${INTERSHEET_REFS}"
-			(at 72.9125 121.92 0)
+			(at 52.5925 121.92 0)
 			(hide yes)
 			(show_name no)
@@
 	(global_label "uC_CAN_TX0"
 		(shape input)
-		(at 87.63 119.38 180)
+		(at 67.31 119.38 180)
 		(fields_autoplaced yes)
 		(effects
@@
 		)
 		(property "Intersheetrefs" "${INTERSHEET_REFS}"
-			(at 73.2149 119.38 0)
+			(at 52.8949 119.38 0)
 			(hide yes)
 			(show_name no)
